File: kicad/JoySpeak.kicad_sch (KiCad schematic)
At the start: 18 parts, among them CN1 AUDIO_IN, CN2 AUDIO_OUT, J2 Hexpansion-Connector, SW3 TS-1187A-B-A-B, SW4 TS-1187A-B-A-B, U1 TLV320AIC3100IRHBR, U2 YV13S-L7.85-B10KA(60)-0-DL01, U3 SN65HVD230, U4 RP2040-ZERO

Commit message: Commiting before simplification
Parts:
- removed C1, C2: 1uF-10V, Capacitor_SMD:C_0603_1608Metric_Pad1.08x0.95mm_HandSolder, symbol Device:C
- removed D1, D2, D3: LED, symbol Device:LED
- removed RJ1, RJ2: R-RJ45R08P-A004, lcsc_footprints:C385834_RJ45-TH_R-RJ45R08P-A004, symbol lcsc_imported:R-RJ45R08P-A004
- removed U1: TLV320AIC3100IRHBR, lcsc_footprints:C478458_QFN-32_L5_0-W5_0-P0_50-TL-EP3_5, symbol lcsc_imported:TLV320AIC3100IRHBR
- removed U3: SN65HVD230, Package_SO:SOIC-8_3.9x4.9mm_P1.27mm, symbol Interface_CAN_LIN:SN65HVD230
- added C15, C40, C45, C46, C47, C50, C51: 1uF, Capacitor_SMD:C_1206_3216Metric_Pad1.33x1.80mm_HandSolder, symbol Device:C
- added C22, C24, C26, C28: 10uF, Capacitor_SMD:C_1206_3216Metric_Pad1.33x1.80mm_HandSolder, symbol Device:C
- added C23, C25, C27, C29, C30, C31, C34, C35, C37, C39, C41, C42, C43, C44, C48: 100nF, Capacitor_SMD:C_1206_3216Metric_Pad1.33x1.80mm_HandSolder, symbol Device:C
- added C32, C33, C38, C49: 22u, Capacitor_SMD:C_0805_2012Metric_Pad1.18x1.45mm_HandSolder, symbol Device:C
- added D1: MBR0520, Diode_SMD:D_SOD-123, symbol Diode:MBR0520
- added FB2, FB3: MPZ1608S121ATAH0, Inductor_SMD:L_0603_1608Metric, symbol Device:FerriteBead
- added H1, H2: MountingHole_Pad, MountingHole:MountingHole_2.2mm_M2_Pad_Via, symbol Mechanical:MountingHole_Pad
- added J2: Conn_01x05_Pin, lcsc_footprints:HexpansionPads1x05, symbol Connector:Conn_01x05_Pin
- added J3: Conn_01x03_Pin, lcsc_footprints:HexpansionPads1x03, symbol Connector:Conn_01x03_Pin
- added J4: Conn_01x01_Pin, lcsc_footprints:HexpansionPads1x01, symbol Connector:Conn_01x01_Pin
- added JP1: SolderJumper_2_Open, Jumper:SolderJumper-2_P1.3mm_Open_RoundedPad1.0x1.5mm, symbol Jumper:SolderJumper_2_Open
- added LED1, LED2: SK6812MINI-EA, lcsc_footprints:C5378731_LED-SMD_4P-L3_2-W2_8_SK6812MINI-EA, symbol lcsc_imported:SK6812MINI-EA
- added R1: 470R, Resistor_SMD:R_0805_2012Metric_Pad1.20x1.40mm_HandSolder, symbol Device:R
- added R2, R3, R4, R5: 4.7k, Resistor_SMD:R_1206_3216Metric_Pad1.30x1.75mm_HandSolder, symbol Device:R
- added R6: 10k, Resistor_SMD:R_1206_3216Metric_Pad1.30x1.75mm_HandSolder, symbol Device:R
- added R7, R8: 470R, Resistor_SMD:R_1206_3216Metric_Pad1.30x1.75mm_HandSolder, symbol Device:R
- added R9: 47k, Resistor_SMD:R_1206_3216Metric_Pad1.30x1.75mm_HandSolder, symbol Device:R
- added RJ1: HC-RJ45-5JA-2-6-S, lcsc_footprints:C5341200_RJ45-TH_HC-RJ45-5JA-2-6-S, symbol lcsc_imported:HC-RJ45-5JA-2-6-S
- added U1: TLV320AIC3100, Package_DFN_QFN:VQFN-32-1EP_5x5mm_P0.5mm_EP3.5x3.5mm, symbol Audio:TLV320AIC3100
- added U4: AMS1117-1.8, Package_TO_SOT_SMD:SOT-223-3_TabPin2, symbol Regulator_Linear:AMS1117-1.8
- added U6, U7, U8: TPMAX40200AUK+T, lcsc_footprints:C47118006_SOT-23-5_L2_9-W1_6-P0_95-LS2_8-BR_1, symbol lcsc_imported:TPMAX40200AUK+T
- LS1: footprint Connector_PinHeader_2.54mm:PinHeader_1x02_P2.54mm_Vertical -> lcsc_footprints:Speaker_FS2828DS0430-H13.0; now left out of the parts list
- renumbered J2 to J1, SW3 to SW1, SW4 to SW2, U4 to U3
Connections:
- net CAN_RX is gone; now on net HEX_HS_F: U3.2 (GP1)
- net CAN_TX is gone; now on net JOY_BUT: U3.1 (GP0)
- net +3V3_A: now also U2.3 (R1), U2.4 (R2), C15.1, C22.1, C23.1, C24.1, C25.1, FB2.2, U1.17 (AVDD), U1.28 (HPVDD), U4.3 (VI), U8.1 (VDD), U8.3 (EN)
- net +5V: now also C32.1, C33.1, C34.1, C35.1, C44.1, C51.1, D1.2 (A), U7.3 (EN), U7.5 (OUT)
- net AUD_BCLK: now also U1.7 (BCLK)
- net AUD_DIN: now also U1.5 (DIN)
- net AUD_DOUT: now also U1.4 (DOUT)
- net AUD_I2C0_SCL: now also R3.2, U1.10 (SCL)
- net AUD_I2C0_SDA: now also R2.2, U1.9 (SDA)
- net AUD_IN_L: now also C46.2, U1.13 (MIC1LP); no longer CN1.1
- net AUD_IN_R: now also C47.2, U1.14 (MIC1RP); no longer CN1.2
- net AUD_MCLK: now also U1.8 (MCLK)
- net AUD_OUT_L: now also CN2.4, U1.27 (HPL); no longer CN2.1
- net AUD_OUT_R: now also CN2.3, U1.30 (HPR); no longer CN2.2
- net AUD_WCLK: now also U1.6 (WCLK)
- net GND: now also CN1.1, CN1.2, CN2.1, CN2.2, J1.1 (GND), J1.10 (GND), J1.11 (GND), J1.14 (GND), J1.17 (GND), J1.20 (GND), J1.6 (HEXP_DET), U2.11 (SHELL), U2.7 (S1), U2.8 (S2), C15.2, C22.2, C23.2, C24.2, C25.2, C26.2, C27.2, C28.2, C29.2, C30.1, C31.2, C32.2, C33.2, C34.2, C35.2, C37.2, C38.2, C39.2, C40.2, C41.1, C42.1, C44.2, C48.2, C49.2, C50.2, C51.2, H1.1, H2.1, LED1.3 (GND), LED2.3 (GND), R9.2, RJ1.11, RJ1.13, RJ1.14, RJ1.3, RJ1.5, RJ1.6, U1.1 (IOVSS), U1.16 (AVSS), U1.18 (DVSS), U1.20 (SPKVSS), U1.25 (SPKVSS), U1.29 (HPVSS), U1.33 (EP), U4.1 (GND), U6.2 (GND), U7.2 (GND), U8.2 (GND)
- net HEX_I2C1_SDA: now also U3.7 (GP6), R4.2; no longer U3.3 (GP2)
- net JOY_ADC0: now also C42.2, C43.1, R8.2; no longer U2.2 (R1)
- net JOY_ADC1: now also C41.2, R7.1; no longer U2.5 (R2)
- net MEMS_MIC: now also C45.1, U1.15 (MIC1LM); no longer MIC1.1 (OUT)
- net MICBIAS: now also C31.1, C40.1, FB3.2, U1.12 (MICBIAS)
- net RESETN: now also U3.9 (GP8), C30.2, R6.1, U1.31 (~{RESET})
- net SPK+: now also U1.22 (SPKP), U1.26 (SPKP)
- net SPK-: now also U1.19 (SPKM), U1.23 (SPKM)
- net JACK_OUT_DETECT: now reaches CN2.6
- net JACK_OUT_DETECT: now also U3.4 (GP3)
- net JOY_BUT: now reaches U2.10 (S4)
- net JOY_BUT: now also U2.9 (S3)
- net at MIC1.4 (VDD): now also FB3.1
- net at CN1.3: now also C47.1
- net at CN1.4: now also C46.1
- net JACK_IN_DETECT: now reaches CN1.6
- net JACK_IN_DETECT: now also U3.3 (GP2)
- net LEDS_DIN: now reaches U3.10 (GP9)
- net LEDS_DIN: now also R1.1
- net PJON_DATA: now reaches U3.16 (GP15)
- net PJON_DATA: now also R9.1, RJ1.12, RJ1.4
- net HEX_I2C1_SCL: now reaches U3.8 (GP7)
- net HEX_I2C1_SCL: now also J1.5 (SCL), R5.2
- net HEX_HS_F: now reaches J1.12 (HS_F)
- net at J1.13 (HS_G): now also J3.1 (Pin_1)
- net at J1.15 (3V3), J1.16 (3V3): now also C38.1, C39.1, U6.1 (VDD)
- net at J1.18 (HS_H): now also J3.2 (Pin_2)
- net at J1.19 (HS_I): now also J3.3 (Pin_3)
- net at J1.2 (LS_A): now also J2.1 (Pin_1)
- net at J1.3 (LS_B): now also J2.2 (Pin_2)
- net at J1.7 (LS_C): now also J2.3 (Pin_3)
- net at J1.8 (LS_D): now also J2.4 (Pin_4)
- net at J1.9 (LS_E): now also J2.5 (Pin_5)
- removed net +3V3: U2.3 (R1), U2.4 (R2), U3.21 (3V3)
- removed net HEX_I2C0_SCL: J1.5 (SCL), U3.4 (GP3)
- new net: LED1.4 (DIN), R1.2
- new net: C48.1, C49.1, RJ1.1, RJ1.10, RJ1.2, RJ1.9, U7.1 (VDD)
- new net: R8.1, U2.2 (R1)
- new net: D1.1 (K), U1.21 (SPKVDD), U1.24 (SPKVDD), U8.5 (OUT)
- new net: JP1.1 (A), U1.11 (VOL/MICDET)
- new net: C43.2, JP1.2 (B)
- new net: C45.2, MIC1.1 (OUT)
- new net: J4.1 (Pin_1), U1.32 (GPIO1)
- new net: R7.2, U2.5 (R2)
- new net: LED1.2 (DOUT), LED2.4 (DIN)
- new net +1V8: C28.1, C29.1, U1.3 (DVDD), U4.2 (VO)
- new net +3V3_D: C26.1, C27.1, C37.1, C50.1, FB2.1, LED1.1 (VDD), LED2.1 (VDD), R2.1, R3.1, R4.1, R5.1, R6.2, U1.2 (IOVDD), U3.21 (3V3), U6.3 (EN), U6.5 (OUT)
- no-connect marks 17 -> 14
Other:
- note added: "1 x bulk 2 x noise protection"
- note added: "5V"
- note added: "AVDD"
- note added: "AVSS"
- note added: "DC-Blocking Cap"
- note added: "DVDD"
- note added: "HPVDD"
- note added: "IOVDD"
- note added: "Reference https://github.com/aitesam961/OpenADSP"
- note added: "SPKVDD"
- note added: "Use X7R/X5R ceramic dielectrics 16V to handle 5V"
- note added: "VR1 (VERTICAL)"
- note added: "VR2 (HORIZONAL)"
- moved on the sheet: CN1, CN2, J1, LS1, MIC1, SW1, SW2, U2, U3

Commit message: Started jumpering power. Consolidated cap and resistor values
Parts:
- removed C48: 100nF, Capacitor_SMD:C_1206_3216Metric_Pad1.33x1.80mm_HandSolder, symbol Device:C
- removed C49: 22u, Capacitor_SMD:C_0805_2012Metric_Pad1.18x1.45mm_HandSolder, symbol Device:C
- removed C50, C51: 1uF, Capacitor_SMD:C_1206_3216Metric_Pad1.33x1.80mm_HandSolder, symbol Device:C
- removed D1: MBR0520, Diode_SMD:D_SOD-123, symbol Diode:MBR0520
- removed R6: 10k, Resistor_SMD:R_1206_3216Metric_Pad1.30x1.75mm_HandSolder, symbol Device:R
- removed U6, U7, U8: TPMAX40200AUK+T, lcsc_footprints:C47118006_SOT-23-5_L2_9-W1_6-P0_95-LS2_8-BR_1, symbol lcsc_imported:TPMAX40200AUK+T
- added JP2: RP2040_Voltage_Jumper, Connector_PinHeader_2.54mm:PinHeader_1x03_P2.54mm_Vertical, symbol Jumper:Jumper_3_Open
- added JP3: Jumper_3_Open, Connector_PinHeader_2.54mm:PinHeader_1x03_P2.54mm_Vertical, symbol Jumper:Jumper_3_Open
- added JP4: Speaker_Voltage_Jumper, Connector_PinHeader_2.54mm:PinHeader_1x03_P2.54mm_Vertical, symbol Jumper:Jumper_3_Open
- added R10: 4.7k, Resistor_SMD:R_1206_3216Metric_Pad1.30x1.75mm_HandSolder, symbol Device:R
- C15, C40, C45, C46, C47: value 1uF -> 10uF; LCSC C1848 -> C13585
- C32, C33, C38: value 22u -> 10uF; footprint Capacitor_SMD:C_0805_2012Metric_Pad1.18x1.45mm_HandSolder -> Capacitor_SMD:C_1206_3216Metric_Pad1.33x1.80mm_HandSolder; LCSC C12891 -> C13585
- R1: footprint Resistor_SMD:R_0805_2012Metric_Pad1.20x1.40mm_HandSolder -> Resistor_SMD:R_1206_3216Metric_Pad1.30x1.75mm_HandSolder
Connections:
- net +3V3_D: now also JP3.2 (C), R10.1; no longer U3.21 (3V3)
- net +5V: now also JP2.2 (C); no longer C32.1, C34.1, C44.1, U3.23 (5V)
- net RESETN: now also R10.2
- net +5V_EXTERNAL: now reaches RJ1.1, RJ1.10, RJ1.2, RJ1.9
- net +5V_EXTERNAL: now also JP2.3 (B)
- net SPKVDD: now reaches U1.21 (SPKVDD), U1.24 (SPKVDD)
- net SPKVDD: now also C32.1, C34.1, C44.1, JP4.2 (C)
- net +3V3_TILDAGON: now reaches C38.1, C39.1, J1.15 (3V3), J1.16 (3V3)
- net +3V3_TILDAGON: now also JP3.3 (B), JP4.3 (B)
- new net +3V3_RP2040ZERO: JP3.1 (A), U3.21 (3V3)
- new net +5V_RP2040ZERO: JP2.1 (A), JP4.1 (A), U3.23 (5V)
- no-connect marks 14 -> 11
Other:
- moved on the sheet: RJ1
